Commit message: wip: update xacro files for gazebo garden and rviz2

File: p3dx_description/urdf/p3dx/pioneer3dx.xacro (robot description, xacro)
@@ -1,19 +1,34 @@
 <?xml version="1.0"?>
-<robot xmlns:xacro="http://ros.org/wiki/xacro" name="pioneer3dx" >
+<robot xmlns:xacro="http://ros.org/wiki/xacro" name="pioneer3dx">
   <!-- Obtain launch file arguements -->
-  <xacro:arg name="robot_namespace" default="/"/>
+  <xacro:arg name="robot_namespace" default="/" />
+  <xacro:arg name="camera_enabled" default="true" />
+  <xacro:arg name="lidar_enabled" default="true" />
+  <xacro:arg name="odometry_source" default="encoders" />
   <!-- Import Rviz colors -->
   <xacro:include filename="$(find p3dx_description)/urdf/materials.xacro" />
   <!-- Import robot -->
-  <xacro:include filename="$(find p3dx_description)/urdf/p3dx/pioneer3dx_body.xacro"/>
-  <xacro:pioneer3dx_body name="chassis" parent="base_link" meshes="package://p3dx_description/meshes/p3dx" robot_namespace="$(arg robot_namespace)"/>
+  <xacro:include filename="$(find p3dx_description)/urdf/p3dx/pioneer3dx_body.xacro" />
+  <xacro:pioneer3dx_body name="chassis" parent="base_link"
+    meshes="file://$(find p3dx_description)/meshes/p3dx" robot_namespace="$(arg robot_namespace)"
+    odometry_source="$(arg odometry_source)" />
   <!-- Laser  -->
-  <xacro:include filename="$(find p3dx_description)/urdf/laser/hokuyo.xacro"/>
-  <xacro:laser name="laser" parent="chassis" xyz="0.16 0 0.1" rpy="0 0 0" meshes="package://p3dx_description/meshes/laser" robot_namespace="$(arg robot_namespace)"/>
+  <xacro:if value="$(arg lidar_enabled)">
+    <xacro:include filename="$(find p3dx_description)/urdf/laser/hokuyo.xacro" />
+    <xacro:laser name="laser" parent="chassis" xyz="0.16 0 0.1" rpy="0 0 0"
+      meshes="file://$(find p3dx_description)/meshes/laser" robot_namespace="$(arg robot_namespace)"
+      gpu="true" />
+  </xacro:if>
   <!-- GPU Laser -->
-<!--  <xacro:include filename="$(find description_plugins)/test/multi_robot_scenario/urdf/laser/hokuyo_gpu.xacro"/>-->
-  <!--<xacro:laser_gpu name="front_laser2" parent="chassis" xyz="0.16 0 0.1" rpy="0 0 0" meshes="package://description_plugins/test/multi_robot_scenario/meshes/laser" />-->
+  <!--  <xacro:include filename="$(find
+  description_plugins)/test/multi_robot_scenario/urdf/laser/hokuyo_gpu.xacro"/>-->
+  <!--<xacro:laser_gpu
+  name="front_laser2" parent="chassis" xyz="0.16 0 0.1" rpy="0 0 0" meshes="$(find
+  description_plugins/test/multi_robot_scenario/meshes/laser" />-->
   <!-- Camera -->
-  <xacro:include filename="$(find p3dx_description)/urdf/camera/camera.xacro"/>
-  <xacro:cam name="front_camera" parent="chassis" xyz="0 0 0.5" rpy="0 0 0" meshes="package://p3dx_description/meshes/camera" robot_namespace="$(arg robot_namespace)" />
+  <xacro:if value="$(arg camera_enabled)">
+  <xacro:include filename="$(find p3dx_description)/urdf/camera/camera.xacro" />
+  <xacro:cam name="front_camera" parent="chassis" xyz="0 0 0.5" rpy="0 0 0"
+    meshes="file://$(find p3dx_description)/meshes/camera" robot_namespace="$(arg robot_namespace)" />
+  </xacro:if>
 </robot>

File: p3dx_description/urdf/p3dx/pioneer3dx_body.xacro (robot description, xacro)
@@ -1,29 +1,67 @@
 <?xml version="1.0"?>
 <robot xmlns:xacro="http://ros.org/wiki/xacro">
-  <xacro:include filename="inertia_tensors.xacro"/>
-  <xacro:include filename="pioneer3dx_chassis.xacro"/>
-  <xacro:include filename="battery_block.xacro"/>
-  <xacro:include filename="pioneer3dx_wheel.xacro"/>
-  <xacro:include filename="pioneer3dx_swivel.xacro"/>
-  <xacro:include filename="pioneer3dx_sonar.xacro"/>
-  <xacro:include filename="pioneer3dx_plugins.xacro"/>
-  <xacro:pioneer3dx_plugins robot_namespace="$(arg robot_namespace)"/>
-  <xacro:macro name="pioneer3dx_body" params="name parent meshes robot_namespace">
+  <xacro:include filename="inertia_tensors.xacro" />
+  <xacro:include filename="pioneer3dx_chassis.xacro" />
+  <xacro:include filename="battery_block.xacro" />
+  <xacro:include filename="pioneer3dx_wheel.xacro" />
+  <xacro:include filename="pioneer3dx_swivel.xacro" />
+  <xacro:include filename="pioneer3dx_sonar.xacro" />
+  <xacro:include filename="pioneer3dx_plugins.xacro" />
+  <xacro:pioneer3dx_plugins robot_namespace="$(arg robot_namespace)" />
+  <xacro:macro name="pioneer3dx_body"
+    params="name parent meshes robot_namespace odometry_source:=encoders">
     <!-- base_link -->
-    <link name="${parent}"/>
+    <link name="${parent}" />
     <!-- Chassis -->
-    <xacro:pioneer_chassis name="${name}" parent="base_link" xyz="0 0 0" rpy="0 0 0"  meshes="${meshes}"/>
+    <xacro:pioneer_chassis name="${name}" parent="${parent}" xyz="0 0 0" rpy="0 0 0"
+      meshes="${meshes}" />
     <!-- Front Sonar -->
-    <xacro:pioneer_sonar name="sonar" parent="${name}" xyz="0.109 0 0.209" rpy="0 0 0"  meshes="${meshes}"/>
-    <!-- Akku0 -->
-    <xacro:battery_block name="battery0" parent="${name}" x="-0.14" y="0.00"  z="0.13" mass="2.5" />
+    <xacro:pioneer_sonar name="sonar" parent="${name}" xyz="0.109 0 0.209" rpy="0 0 0"
+      meshes="${meshes}" />
+    <!-- Simulate battery, not in use -->
+    <xacro:battery_block name="battery0" parent="${name}" x="-0.14" y="0.00" z="0.13" mass="2.5" />
     <!-- Wheels -->
-    <xacro:pioneer_wheel side="right" parent="${name}"  xyz="0 -0.15 0.09" rpy="0 0 0" radius="0.09" meshes="${meshes}"/>
-    <xacro:pioneer_wheel side="left"  parent="${name}"  xyz="0 0.15 0.09" rpy="0 0 0" radius="0.09" meshes="${meshes}"/>
-    <xacro:pioneer_swivel parent="${name}"  xyz="-0.185 0 0.055" rpy="0 0 0" meshes="${meshes}"/>
+    <xacro:pioneer_wheel side="right" parent="${name}" xyz="0 -0.15 0.09" rpy="0 0 0" radius="0.09"
+      meshes="${meshes}" />
+    <xacro:pioneer_wheel side="left" parent="${name}" xyz="0 0.15 0.09" rpy="0 0 0" radius="0.09"
+      meshes="${meshes}" />
+    <xacro:pioneer_swivel parent="${name}" xyz="-0.185 0 0.055" rpy="0 0 0" meshes="${meshes}" />
     <!-- Motor plugin -->
-    <!-- <xacro:pioneer3dx_diff_drive /> -->
+    <gazebo>
+      <plugin filename="ignition-gazebo-diff-drive-system"
+        name="ignition::gazebo::systems::DiffDrive">
+        <left_joint>left_hub_joint</left_joint>
+        <right_joint>right_hub_joint</right_joint>
+        <wheel_separation>${0.3 + 0.01}</wheel_separation>
+        <wheel_radius>${0.09+0.01}</wheel_radius>
+        <odom_publish_frequency>50</odom_publish_frequency>
+        <topic>RosAria/cmd_vel</topic>
+        <xacro:if value="${odometry_source == 'encoders'}">
+          <odom_topic>RosAria/odom</odom_topic>
+          <tf_topic>/tf</tf_topic>
+        </xacro:if>
+        <frame_id>odom</frame_id>
+        <child_frame_id>base_link</child_frame_id>
+      </plugin>
+    </gazebo>
+    <xacro:if value="${odometry_source == 'world'}">
+      <gazebo>
+        <plugin filename="libignition-gazebo6-odometry-publisher-system"
+          name="ignition::gazebo::systems::OdometryPublisher">
+          <odom_frame>odom</odom_frame>
+          <robot_base_frame>base_link</robot_base_frame>
+          <odom_topic>RosAria/odom</odom_topic>
+          <tf_topic>/tf</tf_topic>
+          <dimensions>2</dimensions>
+          <odom_publish_frequency>50</odom_publish_frequency>
+        </plugin>
+      </gazebo>
+    </xacro:if>
     <!-- Joints plugin -->
-    <!-- <xacro:pioneer3dx_joints_state_publisher /> -->
+    <gazebo>
+      <plugin filename="ignition-gazebo-joint-state-publisher-system"
+        name="ignition::gazebo::systems::JointStatePublisher">
+      </plugin>
+    </gazebo>
   </xacro:macro>
 </robot>
