Commit message: wip: update gz plugin for lidar

File: p3dx_description/urdf/laser/hokuyo.xacro (robot description, xacro)
@@ -1,63 +1,96 @@
 <?xml version="1.0"?>
 <robot xmlns:xacro="http://ros.org/wiki/xacro">
-<!-- Front Laser -->
-<xacro:macro name="laser" params="name parent xyz rpy meshes robot_namespace" >
-  <joint name="${parent}_${name}_joint" type="fixed">
+  <!-- Front Laser -->
+  <xacro:macro name="laser" params="gpu:=false name parent xyz rpy meshes robot_namespace">
+    <joint name="${parent}_${name}_joint" type="fixed">
       <axis xyz="0 0 1" />
-      <origin xyz="${xyz}" rpy="${rpy}"/>
-      <parent link="${parent}"/>
-      <child link="${name}"/>
+      <origin xyz="${xyz}" rpy="${rpy}" />
+      <parent link="${parent}" />
+      <child link="${name}" />
     </joint>
     <link name="${name}">
       <collision>
-        <origin xyz="0 0 0" rpy="0 0 0"/>
+        <origin xyz="0 0 0" rpy="0 0 0" />
         <geometry>
-          <box size="0.1 0.1 0.1"/>
+          <box size="0.1 0.1 0.1" />
         </geometry>
       </collision>
       <visual>
-        <origin xyz="0 0 0" rpy="0 0 0"/>
+        <origin xyz="0 0 0" rpy="0 0 0" />
         <geometry>
-          <mesh filename="${meshes}/hokuyo.dae"/>
+          <mesh filename="${meshes}/hokuyo.dae" />
         </geometry>
       </visual>
       <inertial>
         <mass value="1e-5" />
-        <origin xyz="0 0 0" rpy="0 0 0"/>
+        <origin xyz="0 0 0" rpy="0 0 0" />
         <inertia ixx="1e-6" ixy="0" ixz="0" iyy="1e-6" iyz="0" izz="1e-6" />
       </inertial>
     </link>
-    <gazebo reference="${name}">
-        <sensor name="laser" type="ray">
-        <pose>0 0 0 0 0 0</pose>
-          <ray>
+    <plugin filename="ignition-gazebo-sensors-system" name="ignition::gazebo::systems::Sensors">
+      <render_engine>ogre2</render_engine>
+    </plugin>
+    <xacro:if value="${gpu}">
+      <gazebo reference="${name}">
+        <sensor name='gpu_lidar' type='gpu_lidar'>
+          <topic>scan</topic>
+          <update_rate>30</update_rate>
+          <ignition_frame_id>${name}</ignition_frame_id>
+          <lidar>
             <scan>
               <horizontal>
-                <!-- The Hokuyo UTM-30LX-EW Scanning Laser Rangefinder  has  683 steps with 0.35139 Degree resolution -->
+                <samples>683</samples>
                 <resolution>1</resolution>
                 <max_angle>1.8326</max_angle> <!-- 105 Degree -->
                 <min_angle>-1.8326</min_angle> <!-- -105 Degree -->
-                <samples>683</samples>
               </horizontal>
             </scan>
             <range>
               <min>0.08</min>
-              <max>30</max>
+              <max>30.0</max>
               <resolution>0.01</resolution>
             </range>
-          </ray>
-          <plugin name="laser" filename="libgazebo_ros_laser.so" >
-            <robotNamespace>${robot_namespace}</robotNamespace>
-            <topicName>scan</topicName>
-            <frameName>${name}</frameName>
-          </plugin>
-          <!--
-          <plugin name="laser" filename="libRayPlugin.so" />
-          -->
-          <always_on>1</always_on>
-          <update_rate>30</update_rate>
+            <noise>
+              <type>gaussian</type>
+              <mean>0.0</mean>
+              <stddev>0.001</stddev>
+            </noise>
+          </lidar>
+          <alwaysOn>1</alwaysOn>
           <visualize>true</visualize>
         </sensor>
-    </gazebo>
-</xacro:macro>
+      </gazebo>
+    </xacro:if>
+    <xacro:unless value="${gpu}">
+      <gazebo reference="${name}">
+        <sensor name='lidar' type='lidar'>
+          <topic>scan</topic>
+          <update_rate>30</update_rate>
+          <ignition_frame_id>${name}</ignition_frame_id>
+          <lidar>
+            <scan>
+              <horizontal>
+                <samples>683</samples>
+                <resolution>1</resolution>
+                <max_angle>1.8326</max_angle> <!-- 105 Degree -->
+                <min_angle>-1.8326</min_angle> <!-- -105 Degree -->
+              </horizontal>
+            </scan>
+            <range>
+              <min>0.08</min>
+              <max>30.0</max>
+              <resolution>0.01</resolution>
+            </range>
+            <noise>
+              <type>gaussian</type>
+              <mean>0.0</mean>
+              <stddev>0.001</stddev>
+            </noise>
+          </lidar>
+          <alwaysOn>1</alwaysOn>
+          <visualize>true</visualize>
+        </sensor>
+      </gazebo>
+    </xacro:unless>
+  </xacro:macro>
 </robot>

Commit message: wip: let p3dx use full scan instead of -105 to 105 scan

File: p3dx_description/urdf/laser/hokuyo.xacro (robot description, xacro)
@@ -2,5 +2,5 @@
 <robot xmlns:xacro="http://ros.org/wiki/xacro">
   <!-- Front Laser -->
-  <xacro:macro name="laser" params="gpu:=false name parent xyz rpy meshes robot_namespace">
+  <xacro:macro name="laser" params="gpu:=false scan:=scan name parent xyz rpy meshes robot_namespace">
     <joint name="${parent}_${name}_joint" type="fixed">
       <axis xyz="0 0 1" />
@@ -33,7 +33,7 @@
     <xacro:if value="${gpu}">
       <gazebo reference="${name}">
-        <sensor name='gpu_lidar' type='gpu_lidar'>
+        <sensor name='gpu_lidar_${name}' type='gpu_lidar'>
           <xacro:if value="${robot_namespace == '/'}">
-            <topic>scan</topic>
+          <topic>${scan}</topic>
             <gz_frame_id>${name}</gz_frame_id>
           </xacro:if>
@@ -48,6 +48,6 @@
                 <samples>683</samples>
                 <resolution>1</resolution>
-                <max_angle>1.8326</max_angle> <!-- 105 Degree -->
-                <min_angle>-1.8326</min_angle> <!-- -105 Degree -->
+                <max_angle>3.14159</max_angle>
+                <min_angle>-3.14159</min_angle>
               </horizontal>
             </scan>
@@ -70,11 +70,11 @@
     <xacro:unless value="${gpu}">
       <gazebo reference="${name}">
-        <sensor name='lidar' type='lidar'>
+        <sensor name='lidar_${name}' type='lidar'>
           <xacro:if value="${robot_namespace == '/'}">
-            <topic>scan</topic>
+            <topic>${scan}</topic>
             <gz_frame_id>${name}</gz_frame_id>
           </xacro:if>
           <xacro:unless value="${robot_namespace == '/'}">
-            <topic>${robot_namespace}/scan</topic>
+            <topic>${robot_namespace}/${scan}</topic>
             <gz_frame_id>${robot_namespace}/${name}</gz_frame_id>
           </xacro:unless>
@@ -85,6 +85,6 @@
                 <samples>683</samples>
                 <resolution>1</resolution>
-                <max_angle>1.8326</max_angle> <!-- 105 Degree -->
-                <min_angle>-1.8326</min_angle> <!-- -105 Degree -->
+                <max_angle>3.14159</max_angle>
+                <min_angle>-3.14159</min_angle>
               </horizontal>
             </scan>

Commit message: wip: reformat and use gz-sim plugins
Using latest Gazebo Harmonic Eco System!

File: p3dx_description/urdf/laser/hokuyo.xacro (robot description, xacro)
@@ -2,5 +2,6 @@
 <robot xmlns:xacro="http://ros.org/wiki/xacro">
   <!-- Front Laser -->
-  <xacro:macro name="laser" params="gpu:=false scan:=scan name parent xyz rpy meshes robot_namespace">
+  <xacro:macro name="laser"
+    params="gpu:=false scan:=scan name parent xyz rpy meshes robot_namespace">
     <joint name="${parent}_${name}_joint" type="fixed">
       <axis xyz="0 0 1" />
@@ -28,12 +29,12 @@
       </inertial>
     </link>
-    <plugin filename="ignition-gazebo-sensors-system" name="ignition::gazebo::systems::Sensors">
+    <plugin filename="gz-sim-sensors-system" name="gz::sim::systems::Sensors">
       <render_engine>ogre2</render_engine>
     </plugin>
     <xacro:if value="${gpu}">
       <gazebo reference="${name}">
-        <sensor name='gpu_lidar_${name}' type='gpu_lidar'>
+        <sensor name='${name}' type='gpu_lidar'>
           <xacro:if value="${robot_namespace == '/'}">
-          <topic>${scan}</topic>
+            <topic>${scan}</topic>
             <gz_frame_id>${name}</gz_frame_id>
           </xacro:if>
@@ -42,6 +43,7 @@
             <gz_frame_id>${robot_namespace}/${name}</gz_frame_id>
           </xacro:unless>
+          <pose>0 0 0 0 0 0</pose>
           <update_rate>30</update_rate>
-          <lidar>
+          <ray>
             <scan>
               <horizontal>
@@ -62,8 +64,36 @@
               <stddev>0.001</stddev>
             </noise>
-          </lidar>
+          </ray>
           <alwaysOn>1</alwaysOn>
           <visualize>true</visualize>
         </sensor>
+        <!-- <sensor name="hls_lfcd_lds" type="gpu_lidar"> -->
+        <!--   <always_on>true</always_on> -->
+        <!--   <visualize>true</visualize> -->
+        <!--   <pose>-0.064 0 0.15 0 0 0</pose> -->
+        <!--   <update_rate>5</update_rate> -->
+        <!--   <topic>$(arg namespace)/scan</topic> -->
+        <!--   <gz_frame_id>base_scan</gz_frame_id> -->
+        <!--   <ray> -->
+        <!--     <scan> -->
+        <!--       <horizontal> -->
+        <!--         <samples>360</samples> -->
+        <!--         <resolution>1.000000</resolution> -->
+        <!--         <min_angle>0.000000</min_angle> -->
+        <!--         <max_angle>6.280000</max_angle> -->
+        <!--       </horizontal> -->
+        <!--     </scan> -->
+        <!--     <range> -->
+        <!--       <min>0.00001</min> -->
+        <!--       <max>20.0</max> -->
+        <!--       <resolution>0.015000</resolution> -->
+        <!--     </range> -->
+        <!--     <noise> -->
+        <!--       <type>gaussian</type> -->
+        <!--       <mean>0.0</mean> -->
+        <!--       <stddev>0.01</stddev> -->
+        <!--     </noise> -->
+        <!--   </ray> -->
+        <!-- </sensor> -->
       </gazebo>
     </xacro:if>

File: p3dx_description/urdf/p3dx/pioneer3dx.xacro (robot description, xacro)
@@ -28,7 +28,12 @@
   <!-- Camera -->
   <xacro:if value="$(arg camera_enabled)">
-  <xacro:include filename="$(find p3dx_description)/urdf/camera/camera.xacro" />
-  <xacro:cam name="front_camera" parent="chassis" xyz="0 0 0.5" rpy="0 0 0"
-    meshes="file://$(find p3dx_description)/meshes/camera" robot_namespace="$(arg robot_namespace)" />
+    <xacro:include filename="$(find p3dx_description)/urdf/camera/camera.xacro" />
+    <xacro:cam name="front_camera" parent="chassis" xyz="0 0 0.5" rpy="0 0 0"
+      meshes="file://$(find p3dx_description)/meshes/camera"
+      robot_namespace="$(arg robot_namespace)" />
   </xacro:if>
+  <!-- IMU -->
+  <xacro:include filename="$(find p3dx_description)/urdf/imu/imu.xacro" />
+  <xacro:imu_sensor name="imu" parent="chassis" xyz="0 0 0" rpy="0 0 0"
+    robot_namespace="$(arg robot_namespace)" />
 </robot>

File: p3dx_description/urdf/p3dx/pioneer3dx_body.xacro (robot description, xacro)
@@ -27,6 +27,6 @@
     <!-- Motor plugin -->
     <gazebo>
-      <plugin filename="ignition-gazebo-diff-drive-system"
-        name="ignition::gazebo::systems::DiffDrive">
+      <plugin filename="gz-sim-diff-drive-system"
+        name="gz::sim::systems::DiffDrive">
         <left_joint>left_hub_joint</left_joint>
         <right_joint>right_hub_joint</right_joint>
@@ -62,6 +62,6 @@
     <xacro:if value="${odometry_source == 'world'}">
       <gazebo>
-        <plugin filename="libignition-gazebo6-odometry-publisher-system"
-          name="ignition::gazebo::systems::OdometryPublisher">
+        <plugin filename="libgz-sim6-odometry-publisher-system"
+          name="gz::sim::systems::OdometryPublisher">
           <odom_frame>odom</odom_frame>
           <xacro:if value="${robot_namespace == '/'}">
@@ -81,6 +81,6 @@
     <!-- Joints plugin -->
     <gazebo>
-      <plugin filename="ignition-gazebo-joint-state-publisher-system"
-        name="ignition::gazebo::systems::JointStatePublisher">
+      <plugin filename="gz-sim-joint-state-publisher-system"
+        name="gz::sim::systems::JointStatePublisher">
       </plugin>
     </gazebo>
