Commit message: working single robot with namespace

File: p3dx_description/urdf/camera/camera.xacro (robot description, xacro)
@@ -2,5 +2,5 @@
 <robot xmlns:xacro="http://ros.org/wiki/xacro">
 <!-- Camera -->
-<xacro:macro name="cam" params="name parent xyz rpy meshes">
+<xacro:macro name="cam" params="name parent xyz rpy meshes robot_namespace">
   <joint name="${parent}_${name}_joint" type="fixed">
       <axis xyz="0 0 1" />
@@ -58,5 +58,5 @@
       </camera>
       <plugin name="camera_controller" filename="libgazebo_ros_camera.so">
-        <robotNamespace></robotNamespace>
+        <robotNamespace>${robot_namespace}</robotNamespace>
         <alwaysOn>true</alwaysOn>
         <updateRate>0.0</updateRate>

File: p3dx_description/urdf/laser/hokuyo.xacro (robot description, xacro)
@@ -2,5 +2,5 @@
 <robot xmlns:xacro="http://ros.org/wiki/xacro">
 <!-- Front Laser -->
-<xacro:macro name="laser" params="name parent xyz rpy meshes" >
+<xacro:macro name="laser" params="name parent xyz rpy meshes robot_namespace" >
   <joint name="${parent}_${name}_joint" type="fixed">
       <axis xyz="0 0 1" />
@@ -48,5 +48,5 @@
           </ray>
           <plugin name="laser" filename="libgazebo_ros_laser.so" >
-            <robotNamespace></robotNamespace>
+            <robotNamespace>${robot_namespace}</robotNamespace>
             <topicName>scan</topicName>
             <frameName>${name}</frameName>

File: p3dx_description/urdf/p3dx/pioneer3dx.xacro (robot description, xacro)
@@ -1,12 +1,14 @@
 <?xml version="1.0"?>
 <robot xmlns:xacro="http://ros.org/wiki/xacro" name="pioneer3dx" >
+  <!-- Obtain launch file arguements -->
+  <xacro:arg name="robot_namespace" default="/"/>
   <!-- Import Rviz colors -->
   <xacro:include filename="$(find p3dx_description)/urdf/materials.xacro" />
   <!-- Import robot -->
   <xacro:include filename="$(find p3dx_description)/urdf/p3dx/pioneer3dx_body.xacro"/>
-  <xacro:pioneer3dx_body name="chassis" parent="base_link" meshes="package://p3dx_description/meshes/p3dx"/>
+  <xacro:pioneer3dx_body name="chassis" parent="base_link" meshes="package://p3dx_description/meshes/p3dx" robot_namespace="$(arg robot_namespace)"/>
   <!-- Laser  -->
   <xacro:include filename="$(find p3dx_description)/urdf/laser/hokuyo.xacro"/>
-  <xacro:laser name="laser" parent="chassis" xyz="0.16 0 0.1" rpy="0 0 0" meshes="package://p3dx_description/meshes/laser"/>
+  <xacro:laser name="laser" parent="chassis" xyz="0.16 0 0.1" rpy="0 0 0" meshes="package://p3dx_description/meshes/laser" robot_namespace="$(arg robot_namespace)"/>
   <!-- GPU Laser -->
 <!--  <xacro:include filename="$(find description_plugins)/test/multi_robot_scenario/urdf/laser/hokuyo_gpu.xacro"/>-->
@@ -14,4 +16,4 @@
   <!-- Camera -->
   <xacro:include filename="$(find p3dx_description)/urdf/camera/camera.xacro"/>
-  <xacro:cam name="front_camera" parent="chassis" xyz="0 0 0.5" rpy="0 0 0" meshes="package://p3dx_description/meshes/camera" />
+  <xacro:cam name="front_camera" parent="chassis" xyz="0 0 0.5" rpy="0 0 0" meshes="package://p3dx_description/meshes/camera" robot_namespace="$(arg robot_namespace)" />
 </robot>

File: p3dx_description/urdf/p3dx/pioneer3dx_body.xacro (robot description, xacro)
@@ -8,5 +8,6 @@
   <xacro:include filename="pioneer3dx_sonar.xacro"/>
   <xacro:include filename="pioneer3dx_plugins.xacro"/>
-  <xacro:macro name="pioneer3dx_body" params="name parent meshes">
+  <xacro:pioneer3dx_plugins robot_namespace="$(arg robot_namespace)"/>
+  <xacro:macro name="pioneer3dx_body" params="name parent meshes robot_namespace">
     <!-- base_link -->
     <link name="${parent}"/>

File: p3dx_description/urdf/p3dx/pioneer3dx_plugins.xacro (robot description, xacro)
@@ -1,16 +1,18 @@
 <?xml version="1.0"?>
 <robot xmlns:xacro="http://ros.org/wiki/xacro">
-  <gazebo>
-    <plugin name="gazebo_ros_control" filename="libgazebo_ros_control.so">
-        <robotNamespace>$(arg robot_namespace)</robotNamespace>
-    </plugin>
-  </gazebo>
+  <xacro:macro name="pioneer3dx_plugins" params="robot_namespace">
     <gazebo>
-        <plugin name="joint_state_publisher" filename="libgazebo_ros_joint_state_publisher.so">
+      <plugin name="gazebo_ros_control" filename="libgazebo_ros_control.so">
           <robotNamespace>$(arg robot_namespace)</robotNamespace>
-          <jointName>chassis_swivel_joint, swivel_wheel_joint, left_hub_joint, right_hub_joint</jointName>
-          <updateRate>10.0</updateRate>
-          <alwaysOn>true</alwaysOn>
-        </plugin>
+          <legacyModeNS>true</legacyModeNS>
+      </plugin>
     </gazebo>
+      <gazebo>
+          <plugin name="joint_state_publisher" filename="libgazebo_ros_joint_state_publisher.so">
+            <jointName>chassis_swivel_joint, swivel_wheel_joint, left_hub_joint, right_hub_joint</jointName>
+            <updateRate>10.0</updateRate>
+            <alwaysOn>true</alwaysOn>
+          </plugin>
+      </gazebo>
+  </xacro:macro>
 </robot>

Commit message: wip: update gz plugin for cam

File: p3dx_description/urdf/camera/camera.xacro (robot description, xacro)
@@ -1,77 +1,57 @@
 <?xml version="1.0"?>
 <robot xmlns:xacro="http://ros.org/wiki/xacro">
-<!-- Camera -->
-<xacro:macro name="cam" params="name parent xyz rpy meshes robot_namespace">
-  <joint name="${parent}_${name}_joint" type="fixed">
+  <!-- Camera -->
+  <xacro:macro name="cam" params="name parent xyz rpy meshes robot_namespace">
+    <joint name="${parent}_${name}_joint" type="fixed">
       <axis xyz="0 0 1" />
-      <origin xyz="${xyz}" rpy="${rpy}"/>
-      <parent link="${parent}"/>
-      <child link="${name}"/>
-  </joint>
-  <!-- Camera -->
-  <link name="${name}">
-    <inertial>
-      <mass value="1e-5" />
-      <origin xyz="0 0 0" rpy="0 0 0"/>
-      <inertia ixx="1e-6" ixy="0" ixz="0" iyy="1e-6" iyz="0" izz="1e-6" />
-    </inertial>
-    <visual>
-      <origin xyz="0 0 0" rpy="0 1.57 0"/>
-      <geometry>
-        <cylinder radius="0.03" length="0.1"/>
-        <!-- <mesh filename="${meshes}/camera.dae"/> -->
-      </geometry>
-      <material name="grey"/>
-    </visual>
-    <collision>
-      <origin xyz="0 0 0" rpy="0 1.57 0"/>
-      <geometry>
-        <cylinder radius="0.03" length="0.1"/>
-      </geometry>
-    </collision>
-  </link>
-  <gazebo reference="${name}">
-    <material value="Gazebo/Grey"/>
-  </gazebo>
-  <gazebo reference="${name}">
-    <sensor type="camera" name="camera1">
-      <update_rate>30.0</update_rate>
-      <camera name="head">
-        <horizontal_fov>1.3962634</horizontal_fov>
-        <image>
-          <width>800</width>
-          <height>800</height>
-          <format>R8G8B8</format>
-        </image>
-        <clip>
-          <near>0.02</near>
-          <far>300</far>
-        </clip>
-        <noise>
-          <type>gaussian</type>
-          <!-- Noise is sampled independently per pixel on each frame.
-               That pixel's noise value is added to each of its color
-               channels, which at that point lie in the range [0,1]. -->
-          <mean>0.0</mean>
-          <stddev>0.007</stddev>
-        </noise>
-      </camera>
-      <plugin name="camera_controller" filename="libgazebo_ros_camera.so">
-        <robotNamespace>${robot_namespace}</robotNamespace>
-        <alwaysOn>true</alwaysOn>
-        <updateRate>0.0</updateRate>
-        <cameraName>${name}</cameraName>
-        <imageTopicName>image_raw</imageTopicName>
-        <cameraInfoTopicName>camera_info</cameraInfoTopicName>
-        <frameName>${name}</frameName>
-        <hackBaseline>0.07</hackBaseline>
-        <distortionK1>0.0</distortionK1>
-        <distortionK2>0.0</distortionK2>
-        <distortionK3>0.0</distortionK3>
-        <distortionT1>0.0</distortionT1>
-        <distortionT2>0.0</distortionT2>
-      </plugin>
-    </sensor>
-  </gazebo>
-</xacro:macro>
+      <origin xyz="${xyz}" rpy="${rpy}" />
+      <parent link="${parent}" />
+      <child link="${name}" />
+    </joint>
+    <!-- Camera -->
+    <link name="${name}">
+      <inertial>
+        <mass value="1e-5" />
+        <origin xyz="0 0 0" rpy="0 0 0" />
+        <inertia ixx="1e-6" ixy="0" ixz="0" iyy="1e-6" iyz="0" izz="1e-6" />
+      </inertial>
+      <visual>
+        <origin xyz="0 0 0" rpy="0 1.57 0" />
+        <geometry>
+          <cylinder radius="0.03" length="0.1" />
+          <!-- <mesh filename="${meshes}/camera.dae"/> -->
+        </geometry>
+        <material name="grey" />
+      </visual>
+      <collision>
+        <origin xyz="0 0 0" rpy="0 1.57 0" />
+        <geometry>
+          <cylinder radius="0.03" length="0.1" />
+        </geometry>
+      </collision>
+    </link>
+    <gazebo reference="${name}">
+      <material value="Gazebo/Grey" />
+    </gazebo>
+    <gazebo reference="${name}">
+      <sensor type="depth_camera" name="${name}">
+        <update_rate>30.0</update_rate>
+        <topic>${name}</topic>
+        <ignition_frame_id>${name}</ignition_frame_id>
+        <camera_info_topic>${name}/camera_info</camera_info_topic>
+        <camera>
+          <horizontal_fov>1.3962634</horizontal_fov>
+          <image>
+            <width>800</width>
+            <height>800</height>
+            <format>R8G8B8</format>
+          </image>
+          <clip>
+            <near>0.05</near>
+            <far>300</far>
+          </clip>
+        </camera>
+      </sensor>
+    </gazebo>
+  </xacro:macro>
 </robot>
