Commit message: fix: ensure namespace is proper for sensor msgs
/pioneer_a/scan/header has pioneer_a/laser.

File: p3dx_description/urdf/camera/camera.xacro (robot description, xacro)
@@ -1,77 +1,83 @@
 <?xml version="1.0"?>
 <robot xmlns:xacro="http://ros.org/wiki/xacro">
-<!-- Camera -->
-<xacro:macro name="cam" params="name parent xyz rpy meshes robot_namespace">
-  <joint name="${parent}_${name}_joint" type="fixed">
+  <!-- Camera -->
+  <xacro:macro name="cam" params="name parent xyz rpy meshes robot_namespace">
+    <joint name="${parent}_${name}_joint" type="fixed">
       <axis xyz="0 0 1" />
-      <origin xyz="${xyz}" rpy="${rpy}"/>
-      <parent link="${parent}"/>
-      <child link="${name}"/>
-  </joint>
-  <!-- Camera -->
-  <link name="${name}">
-    <inertial>
-      <mass value="1e-5" />
-      <origin xyz="0 0 0" rpy="0 0 0"/>
-      <inertia ixx="1e-6" ixy="0" ixz="0" iyy="1e-6" iyz="0" izz="1e-6" />
-    </inertial>
-    <visual>
-      <origin xyz="0 0 0" rpy="0 1.57 0"/>
-      <geometry>
-        <cylinder radius="0.03" length="0.1"/>
-        <!-- <mesh filename="${meshes}/camera.dae"/> -->
-      </geometry>
-      <material name="grey"/>
-    </visual>
-    <collision>
-      <origin xyz="0 0 0" rpy="0 1.57 0"/>
-      <geometry>
-        <cylinder radius="0.03" length="0.1"/>
-      </geometry>
-    </collision>
-  </link>
-  <gazebo reference="${name}">
-    <material value="Gazebo/Grey"/>
-  </gazebo>
-  <gazebo reference="${name}">
-    <sensor type="camera" name="camera1">
-      <update_rate>30.0</update_rate>
-      <camera name="head">
-        <horizontal_fov>1.3962634</horizontal_fov>
-        <image>
-          <width>800</width>
-          <height>800</height>
-          <format>R8G8B8</format>
-        </image>
-        <clip>
-          <near>0.02</near>
-          <far>300</far>
-        </clip>
-        <noise>
-          <type>gaussian</type>
-          <!-- Noise is sampled independently per pixel on each frame.
+      <origin xyz="${xyz}" rpy="${rpy}" />
+      <parent link="${parent}" />
+      <child link="${name}" />
+    </joint>
+    <!-- Camera -->
+    <link name="${name}">
+      <inertial>
+        <mass value="1e-5" />
+        <origin xyz="0 0 0" rpy="0 0 0" />
+        <inertia ixx="1e-6" ixy="0" ixz="0" iyy="1e-6" iyz="0" izz="1e-6" />
+      </inertial>
+      <visual>
+        <origin xyz="0 0 0" rpy="0 1.57 0" />
+        <geometry>
+          <cylinder radius="0.03" length="0.1" />
+          <!-- <mesh filename="${meshes}/camera.dae"/> -->
+        </geometry>
+        <material name="grey" />
+      </visual>
+      <collision>
+        <origin xyz="0 0 0" rpy="0 1.57 0" />
+        <geometry>
+          <cylinder radius="0.03" length="0.1" />
+        </geometry>
+      </collision>
+    </link>
+    <gazebo reference="${name}">
+      <material value="Gazebo/Grey" />
+    </gazebo>
+    <gazebo reference="${name}">
+      <sensor type="camera" name="camera1">
+        <update_rate>30.0</update_rate>
+        <camera name="head">
+          <horizontal_fov>1.3962634</horizontal_fov>
+          <image>
+            <width>800</width>
+            <height>800</height>
+            <format>R8G8B8</format>
+          </image>
+          <clip>
+            <near>0.02</near>
+            <far>300</far>
+          </clip>
+          <noise>
+            <type>gaussian</type>
+            <!-- Noise is sampled independently per pixel on each frame.
                That pixel's noise value is added to each of its color
                channels, which at that point lie in the range [0,1]. -->
-          <mean>0.0</mean>
-          <stddev>0.007</stddev>
-        </noise>
-      </camera>
-      <plugin name="camera_controller" filename="libgazebo_ros_camera.so">
-        <robotNamespace>${robot_namespace}</robotNamespace>
-        <alwaysOn>true</alwaysOn>
-        <updateRate>0.0</updateRate>
-        <cameraName>${name}</cameraName>
-        <imageTopicName>image_raw</imageTopicName>
-        <cameraInfoTopicName>camera_info</cameraInfoTopicName>
-        <frameName>${name}</frameName>
-        <hackBaseline>0.07</hackBaseline>
-        <distortionK1>0.0</distortionK1>
-        <distortionK2>0.0</distortionK2>
-        <distortionK3>0.0</distortionK3>
-        <distortionT1>0.0</distortionT1>
-        <distortionT2>0.0</distortionT2>
-      </plugin>
-    </sensor>
-  </gazebo>
-</xacro:macro>
+            <mean>0.0</mean>
+            <stddev>0.007</stddev>
+          </noise>
+        </camera>
+        <plugin name="camera_controller" filename="libgazebo_ros_camera.so">
+          <robotNamespace>${robot_namespace}</robotNamespace>
+          <alwaysOn>true</alwaysOn>
+          <updateRate>0.0</updateRate>
+          <imageTopicName>image_raw</imageTopicName>
+          <cameraInfoTopicName>camera_info</cameraInfoTopicName>
+          <xacro:if value="${robot_namespace != '/'}">
+            <cameraName>${robot_namespace}/${name}</cameraName>
+            <frameName>${robot_namespace}/${name}</frameName>
+          </xacro:if>
+          <xacro:unless value="${robot_namespace != '/'}">
+            <cameraName>${name}</cameraName>
+            <frameName>${name}</frameName>
+          </xacro:unless>
+          <hackBaseline>0.07</hackBaseline>
+          <distortionK1>0.0</distortionK1>
+          <distortionK2>0.0</distortionK2>
+          <distortionK3>0.0</distortionK3>
+          <distortionT1>0.0</distortionT1>
+          <distortionT2>0.0</distortionT2>
+        </plugin>
+      </sensor>
+    </gazebo>
+  </xacro:macro>
 </robot>

File: p3dx_description/urdf/laser/hokuyo.xacro (robot description, xacro)
@@ -1,63 +1,66 @@
 <?xml version="1.0"?>
 <robot xmlns:xacro="http://ros.org/wiki/xacro">
-<!-- Front Laser -->
-<xacro:macro name="laser" params="name parent xyz rpy meshes robot_namespace" >
-  <joint name="${parent}_${name}_joint" type="fixed">
+  <!-- Front Laser -->
+  <xacro:macro name="laser" params="name parent xyz rpy meshes robot_namespace">
+    <joint name="${parent}_${name}_joint" type="fixed">
       <axis xyz="0 0 1" />
-      <origin xyz="${xyz}" rpy="${rpy}"/>
-      <parent link="${parent}"/>
-      <child link="${name}"/>
+      <origin xyz="${xyz}" rpy="${rpy}" />
+      <parent link="${parent}" />
+      <child link="${name}" />
     </joint>
     <link name="${name}">
       <collision>
-        <origin xyz="0 0 0" rpy="0 0 0"/>
+        <origin xyz="0 0 0" rpy="0 0 0" />
         <geometry>
-          <box size="0.1 0.1 0.1"/>
+          <box size="0.1 0.1 0.1" />
         </geometry>
       </collision>
       <visual>
-        <origin xyz="0 0 0" rpy="0 0 0"/>
+        <origin xyz="0 0 0" rpy="0 0 0" />
         <geometry>
-          <mesh filename="${meshes}/hokuyo.dae"/>
+          <mesh filename="${meshes}/hokuyo.dae" />
         </geometry>
       </visual>
       <inertial>
         <mass value="1e-5" />
-        <origin xyz="0 0 0" rpy="0 0 0"/>
+        <origin xyz="0 0 0" rpy="0 0 0" />
         <inertia ixx="1e-6" ixy="0" ixz="0" iyy="1e-6" iyz="0" izz="1e-6" />
       </inertial>
     </link>
     <gazebo reference="${name}">
-        <sensor name="laser" type="ray">
+      <sensor name="laser" type="ray">
         <pose>0 0 0 0 0 0</pose>
-          <ray>
-            <scan>
-              <horizontal>
-                <!-- The Hokuyo UTM-30LX-EW Scanning Laser Rangefinder  has  683 steps with 0.35139 Degree resolution -->
-                <resolution>1</resolution>
-                <max_angle>1.8326</max_angle> <!-- 105 Degree -->
-                <min_angle>-1.8326</min_angle> <!-- -105 Degree -->
-                <samples>683</samples>
-              </horizontal>
-            </scan>
-            <range>
-              <min>0.08</min>
-              <max>30</max>
-              <resolution>0.01</resolution>
-            </range>
-          </ray>
-          <plugin name="laser" filename="libgazebo_ros_laser.so" >
-            <robotNamespace>${robot_namespace}</robotNamespace>
-            <topicName>scan</topicName>
+        <ray>
+          <scan>
+            <horizontal>
+              <!-- The Hokuyo UTM-30LX-EW Scanning Laser Rangefinder  has  683 steps with 0.35139
+              Degree resolution -->
+              <resolution>1</resolution>
+              <max_angle>1.8326</max_angle> <!-- 105 Degree -->
+              <min_angle>-1.8326</min_angle> <!-- -105 Degree -->
+              <samples>683</samples>
+            </horizontal>
+          </scan>
+          <range>
+            <min>0.08</min>
+            <max>30</max>
+            <resolution>0.01</resolution>
+          </range>
+        </ray>
+        <plugin name="laser" filename="libgazebo_ros_laser.so">
+          <robotNamespace>${robot_namespace}</robotNamespace>
+          <topicName>scan</topicName>
+          <xacro:if value="${robot_namespace != '/'}">
+            <frameName>${robot_namespace}/${name}</frameName>
+          </xacro:if>
+          <xacro:unless value="${robot_namespace != '/'}">
             <frameName>${name}</frameName>
-          </plugin>
-          <!--
-          <plugin name="laser" filename="libRayPlugin.so" />
-          -->
-          <always_on>1</always_on>
-          <update_rate>30</update_rate>
-          <visualize>true</visualize>
-        </sensor>
+          </xacro:unless>
+        </plugin>
+        <always_on>1</always_on>
+        <update_rate>30</update_rate>
+        <visualize>true</visualize>
+      </sensor>
     </gazebo>
-</xacro:macro>
+  </xacro:macro>
 </robot>

File: p3dx_description/urdf/laser/hokuyo_gpu.xacro (robot description, xacro)
@@ -1,71 +1,76 @@
 <?xml version="1.0"?>
 <robot xmlns:xacro="http://ros.org/wiki/xacro">
-<!-- Front Laser -->
-<xacro:macro name="laser_gpu" params="name parent xyz rpy meshes" >
-  <joint name="${parent}_${name}_joint" type="fixed">
+  <!-- Front Laser -->
+  <xacro:macro name="laser_gpu" params="name parent xyz rpy meshes robot_namespace">
+    <joint name="${parent}_${name}_joint" type="fixed">
       <axis xyz="0 0 1" />
-      <origin xyz="${xyz}" rpy="${rpy}"/>
-      <parent link="${parent}"/>
-      <child link="${name}"/>
+      <origin xyz="${xyz}" rpy="${rpy}" />
+      <parent link="${parent}" />
+      <child link="${name}" />
     </joint>
     <link name="${name}">
       <collision>
-        <origin xyz="0 0 0" rpy="0 0 0"/>
+        <origin xyz="0 0 0" rpy="0 0 0" />
         <geometry>
-          <box size="0.1 0.1 0.1"/>
+          <box size="0.1 0.1 0.1" />
         </geometry>
       </collision>
       <visual>
-        <origin xyz="0 0 0" rpy="0 0 0"/>
+        <origin xyz="0 0 0" rpy="0 0 0" />
         <geometry>
-          <mesh filename="${meshes}/hokuyo.dae"/>
+          <mesh filename="${meshes}/hokuyo.dae" />
         </geometry>
       </visual>
       <inertial>
         <mass value="1e-5" />
-        <origin xyz="0 0 0" rpy="0 0 0"/>
+        <origin xyz="0 0 0" rpy="0 0 0" />
         <inertia ixx="1e-6" ixy="0" ixz="0" iyy="1e-6" iyz="0" izz="1e-6" />
       </inertial>
     </link>
     <gazebo reference="${name}">
-    <sensor type="gpu_ray" name="head_hokuyo_sensor">
-      <pose>0 0 0 0 0 0</pose>
-      <always_on>1</always_on>
-      <update_rate>30</update_rate>
-      <visualize>true</visualize>
-      <ray>
-        <scan>
-          <horizontal>
-            <!-- The URG-04LX-UG01  has  683 steps with 0.35139 Degree resolution -->
-            <resolution>1</resolution>
-            <max_angle>2.0944</max_angle> <!-- 120 Degree -->
-            <min_angle>-2.0944</min_angle> <!-- -120 Degree -->
-            <!--max_angle>3.14</max_angle--> <!-- 120 Degree -->
-            <!--min_angle>-3.14</min_angle--> <!-- -120 Degree -->
-            <samples>683</samples>
-          </horizontal>
-        </scan>
-        <range>
-          <min>0.10</min>
-          <max>140.0</max>
-          <resolution>0.01</resolution>
-        </range>
-        <noise>
-          <type>gaussian</type>
-          <!-- Noise parameters based on published spec for Hokuyo laser
+      <sensor type="gpu_ray" name="head_hokuyo_sensor">
+        <pose>0 0 0 0 0 0</pose>
+        <always_on>1</always_on>
+        <update_rate>30</update_rate>
+        <visualize>true</visualize>
+        <ray>
+          <scan>
+            <horizontal>
+              <!-- The URG-04LX-UG01  has  683 steps with 0.35139 Degree resolution -->
+              <resolution>1</resolution>
+              <max_angle>2.0944</max_angle> <!-- 120 Degree -->
+              <min_angle>-2.0944</min_angle> <!-- -120 Degree -->
+              <!--max_angle>3.14</max_angle--> <!-- 120 Degree -->
+              <!--min_angle>-3.14</min_angle--> <!-- -120 Degree -->
+              <samples>683</samples>
+            </horizontal>
+          </scan>
+          <range>
+            <min>0.10</min>
+            <max>140.0</max>
+            <resolution>0.01</resolution>
+          </range>
+          <noise>
+            <type>gaussian</type>
+            <!-- Noise parameters based on published spec for Hokuyo laser
                achieving "+-30mm" accuracy at range < 10m.  A mean of 0.0m and
                stddev of 0.01m will put 99.7% of samples within 0.03m of the true
                reading. -->
-          <mean>0.0</mean>
-          <stddev>0.01</stddev>
-        </noise>
-      </ray>
-      <plugin name="gazebo_ros_head_hokuyo_controller" filename="libgazebo_ros_gpu_laser.so">
-        <robotNamespace></robotNamespace>
-        <topicName>${name}/scan</topicName>
-        <frameName>${name}</frameName>
-      </plugin>
-    </sensor>
+            <mean>0.0</mean>
+            <stddev>0.01</stddev>
+          </noise>
+        </ray>
+        <plugin name="gazebo_ros_head_hokuyo_controller" filename="libgazebo_ros_gpu_laser.so">
+          <robotNamespace>${robot_namespace}</robotNamespace>
+          <topicName>scan</topicName>
+          <xacro:if value="${robot_namespace != '/'}">
+            <frameName>${robot_namespace}/${name}</frameName>
+          </xacro:if>
+          <xacro:unless value="${robot_namespace != '/'}">
+            <frameName>${name}</frameName>
+          </xacro:unless>
+        </plugin>
+      </sensor>
     </gazebo>
-</xacro:macro>
+  </xacro:macro>
 </robot>

File: p3dx_description/urdf/p3dx/pioneer3dx.xacro (robot description, xacro)
@@ -12,6 +12,6 @@
   <xacro:laser name="laser" parent="chassis" xyz="0.16 0 0.1" rpy="0 0 0" meshes="package://p3dx_description/meshes/laser" robot_namespace="$(arg robot_namespace)"/>
   <!-- GPU Laser -->
-<!--  <xacro:include filename="$(find description_plugins)/test/multi_robot_scenario/urdf/laser/hokuyo_gpu.xacro"/>-->
-  <!--<xacro:laser_gpu name="front_laser2" parent="chassis" xyz="0.16 0 0.1" rpy="0 0 0" meshes="package://description_plugins/test/multi_robot_scenario/meshes/laser" />-->
+  <!-- <xacro:include filename="$(find p3dx_description)/urdf/laser/hokuyo_gpu.xacro"/> -->
+  <!-- <xacro:laser_gpu name="laser" parent="chassis" xyz="0.16 0 0.1" rpy="0 0 0" meshes="package://p3dx_description/meshes/laser" robot_namespace="$(arg robot_namespace)"/> -->
   <!-- Camera -->
   <xacro:include filename="$(find p3dx_description)/urdf/camera/camera.xacro"/>

Commit message: fix: enable camera stream from gazebo

File: p3dx_description/urdf/camera/camera.xacro (robot description, xacro)
@@ -3,5 +3,5 @@
   <!-- Camera -->
   <xacro:macro name="cam" params="name parent xyz rpy meshes robot_namespace">
-    <joint name="${parent}_${name}_joint" type="fixed">
+    <joint name="${name}_joint" type="fixed">
       <axis xyz="0 0 1" />
       <origin xyz="${xyz}" rpy="${rpy}" />
@@ -31,25 +31,39 @@
       </collision>
     </link>
+    <joint name="${name}_optical_joint" type="fixed">
+      <parent link="${name}"/>
+      <child link="${name}_optical"/>
+      <origin xyz="0 0 0" rpy="${-pi/2} 0 ${-pi/2}"/>
+    </joint>
+    <link name="${name}_optical"></link>
     <gazebo reference="${name}">
       <material value="Gazebo/Grey" />
     </gazebo>
     <gazebo reference="${name}">
-      <sensor type="depth_camera" name="${name}">
+      <sensor name="${name}" type="camera">
+        <pose> 0 0 0 0 0 0 </pose>
+        <visualize>true</visualize>
         <update_rate>30.0</update_rate>
-        <topic>${name}</topic>
-        <gz_frame_id>${name}</gz_frame_id>
-        <camera_info_topic>${name}/camera_info</camera_info_topic>
         <camera>
-          <horizontal_fov>1.3962634</horizontal_fov>
-          <image>
-            <width>800</width>
-            <height>800</height>
-            <format>R8G8B8</format>
-          </image>
-          <clip>
-            <near>0.05</near>
-            <far>300</far>
-          </clip>
+          <camera_info_topic>${name}/camera_info</camera_info_topic>
+            <horizontal_fov>1.089</horizontal_fov>
+            <image>
+                <format>R8G8B8</format>
+                <width>640</width>
+                <height>480</height>
+            </image>
+            <clip>
+                <near>0.05</near>
+                <far>8.0</far>
+            </clip>
         </camera>
+        <xacro:if value="${robot_namespace == '/'}">
+          <topic>${name}/image_raw</topic>
+          <gz_frame_id>${name}_optical</gz_frame_id>
+        </xacro:if>
+        <xacro:unless value="${robot_namespace == '/'}">
+        <topic>${robot_namespace}/${name}/image_raw</topic>
+        <gz_frame_id>${robot_namespace}/${name}_optical</gz_frame_id>
+        </xacro:unless>
       </sensor>
     </gazebo>
